Commit message: Linked rviz to gazebo

File: catkin_ws/src/motoman/motoman_hc10_support/urdf/hc10.xacro (robot description, xacro)
@@ -3,3 +3,6 @@
   <xacro:include filename="$(find motoman_hc10_support)/urdf/hc10_macro.xacro" />
   <xacro:motoman_hc10 prefix=""/>
+  <xacro:include filename="$(find motoman_hc10_support)/urdf/joint_motors_macro.xacro"/>
+  <xacro:hc10_gazebo prefix="" />
+  <xacro:hc10_control prefix="" />
 </robot>

File: catkin_ws/src/motoman/motoman_hc10_support/urdf/hc10_macro.xacro (robot description, xacro)
@@ -7,8 +7,8 @@
     <link name="${prefix}base_link">
     	<inertial>
-	   	<origin xyz="0 0 0" rpy="0 0 0"/>
-	   	<mass value="0.1"/>
-	   	<inertia ixx="0.03" ixy="0.03" ixz="0.03" iyy="0.0" iyz="0.0" izz="0.0"/>
-	</inertial>
+        <origin xyz="0 0 0" rpy="0 0 0"/>
+        <mass value="0.1"/>
+        <inertia ixx="0.03" ixy="0.03" ixz="0.03" iyy="0.0" iyz="0.0" izz="0.0"/>
+	    </inertial>
       <visual>
         <geometry>
@@ -25,8 +25,8 @@
     <link name="${prefix}link_1_s">
     	<inertial>
-	   	<origin xyz="0 0 0" rpy="0 0 0"/>
-	   	<mass value="0.1"/>
-	   	<inertia ixx="0.03" ixy="0.03" ixz="0.03" iyy="0.0" iyz="0.0" izz="0.0"/>
-	</inertial>
+        <origin xyz="0 0 0" rpy="0 0 0"/>
+        <mass value="0.1"/>
+        <inertia ixx="0.03" ixy="0.03" ixz="0.03" iyy="0.0" iyz="0.0" izz="0.0"/>
+	    </inertial>
       <visual>
         <geometry>
@@ -43,8 +43,8 @@
     <link name="${prefix}link_2_l">
     	<inertial>
-	   	<origin xyz="0 0 0" rpy="0 0 0"/>
-	   	<mass value="0.1"/>
-	   	<inertia ixx="0.03" ixy="0.03" ixz="0.03" iyy="0.0" iyz="0.0" izz="0.0"/>
-	</inertial>
+        <origin xyz="0 0 0" rpy="0 0 0"/>
+        <mass value="0.1"/>
+        <inertia ixx="0.03" ixy="0.03" ixz="0.03" iyy="0.0" iyz="0.0" izz="0.0"/>
+	    </inertial>
       <visual>
         <geometry>
@@ -61,8 +61,8 @@
     <link name="${prefix}link_3_u">
     	<inertial>
-	   	<origin xyz="0 0 0" rpy="0 0 0"/>
-	   	<mass value="0.1"/>
-	   	<inertia ixx="0.03" ixy="0.03" ixz="0.03" iyy="0.0" iyz="0.0" izz="0.0"/>
-	</inertial>
+        <origin xyz="0 0 0" rpy="0 0 0"/>
+        <mass value="0.1"/>
+        <inertia ixx="0.03" ixy="0.03" ixz="0.03" iyy="0.0" iyz="0.0" izz="0.0"/>
+	    </inertial>
       <visual>
         <geometry>
@@ -79,8 +79,8 @@
     <link name="${prefix}link_4_r">
     	<inertial>
-	   	<origin xyz="0 0 0" rpy="0 0 0"/>
-	   	<mass value="0.1"/>
-	   	<inertia ixx="0.03" ixy="0.03" ixz="0.03" iyy="0.0" iyz="0.0" izz="0.0"/>
-	</inertial>
+        <origin xyz="0 0 0" rpy="0 0 0"/>
+        <mass value="0.1"/>
+        <inertia ixx="0.03" ixy="0.03" ixz="0.03" iyy="0.0" iyz="0.0" izz="0.0"/>
+	    </inertial>
       <visual>
         <geometry>
@@ -97,8 +97,8 @@
     <link name="${prefix}link_5_b">
     	<inertial>
-	   	<origin xyz="0 0 0" rpy="0 0 0"/>
-	   	<mass value="0.1"/>
-	   	<inertia ixx="0.03" ixy="0.03" ixz="0.03" iyy="0.0" iyz="0.0" izz="0.0"/>
-	</inertial>
+        <origin xyz="0 0 0" rpy="0 0 0"/>
+        <mass value="0.1"/>
+        <inertia ixx="0.03" ixy="0.03" ixz="0.03" iyy="0.0" iyz="0.0" izz="0.0"/>
+	    </inertial>
       <visual>
         <geometry>
@@ -115,8 +115,8 @@
     <link name="${prefix}link_6_t">
     	<inertial>
-	   	<origin xyz="0 0 0" rpy="0 0 0"/>
-	   	<mass value="0.1"/>
-	   	<inertia ixx="0.03" ixy="0.03" ixz="0.03" iyy="0.0" iyz="0.0" izz="0.0"/>
-	</inertial>
+        <origin xyz="0 0 0" rpy="0 0 0"/>
+        <mass value="0.1"/>
+        <inertia ixx="0.03" ixy="0.03" ixz="0.03" iyy="0.0" iyz="0.0" izz="0.0"/>
+	    </inertial>
       <visual>
         <geometry>
@@ -133,14 +133,14 @@
     <link name="${prefix}tool0"/>
     	<inertial>
-	   	<origin xyz="0 0 0" rpy="0 0 0"/>
-	   	<mass value="0.1"/>
-	   	<inertia ixx="0.03" ixy="0.03" ixz="0.03" iyy="0.0" iyz="0.0" izz="0.0"/>
-	</inertial>
+        <origin xyz="0 0 0" rpy="0 0 0"/>
+        <mass value="0.1"/>
+        <inertia ixx="0.03" ixy="0.03" ixz="0.03" iyy="0.0" iyz="0.0" izz="0.0"/>
+	    </inertial>
     <!-- end of link list -->
     <!-- joint list -->
     <joint name="world_fixed" type="fixed">
-	   <parent link="world"/>
-	   <child link="${prefix}base"/>
-	</joint>
+	    <parent link="world"/>
+	    <child link="${prefix}base"/>
+	  </joint>
     <joint name="${prefix}joint_1_s" type="revolute">
     	<dynamics damping="1"/>
