Commit message: update urdf and start add camera

File: catkin_ws/src/motoman/motoman_hc10_support/urdf/hc10_macro.xacro (robot description, xacro)
@@ -4,4 +4,5 @@
     <xacro:include filename="$(find motoman_resources)/urdf/common_materials.xacro"/>
     <!-- link list -->
+    <link name="world"/>
     <link name="${prefix}base_link">
       <visual>
@@ -11,4 +12,9 @@
         <xacro:material_yaskawa_blue/>
       </visual>
+      <inertial>
+        <origin xyz="0 0 0" rpy="0 0 0"/>
+        <mass value="0.1"/>
+        <inertia ixx="0.03" ixy="0.03" ixz="0.03" iyy="0.0" iyz="0.0" izz="0.0"/>
+      </inertial>
       <collision>
         <geometry>
@@ -24,4 +30,9 @@
         <xacro:material_yaskawa_blue/>
       </visual>
+      <inertial>
+        <origin xyz="0 0 0" rpy="0 0 0"/>
+        <mass value="0.1"/>
+        <inertia ixx="0.03" ixy="0.03" ixz="0.03" iyy="0.0" iyz="0.0" izz="0.0"/>
+      </inertial>
       <collision>
         <geometry>
@@ -37,4 +48,9 @@
         <xacro:material_yaskawa_blue/>
       </visual>
+      <inertial>
+        <origin xyz="0 0 0" rpy="0 0 0"/>
+        <mass value="0.1"/>
+        <inertia ixx="0.03" ixy="0.03" ixz="0.03" iyy="0.0" iyz="0.0" izz="0.0"/>
+      </inertial>
       <collision>
         <geometry>
@@ -50,4 +66,9 @@
         <xacro:material_yaskawa_blue/>
       </visual>
+      <inertial>
+        <origin xyz="0 0 0" rpy="0 0 0"/>
+        <mass value="0.1"/>
+        <inertia ixx="0.03" ixy="0.03" ixz="0.03" iyy="0.0" iyz="0.0" izz="0.0"/>
+      </inertial>
       <collision>
         <geometry>
@@ -63,4 +84,9 @@
         <xacro:material_yaskawa_blue/>
       </visual>
+      <inertial>
+        <origin xyz="0 0 0" rpy="0 0 0"/>
+        <mass value="0.1"/>
+        <inertia ixx="0.03" ixy="0.03" ixz="0.03" iyy="0.0" iyz="0.0" izz="0.0"/>
+      </inertial>
       <collision>
         <geometry>
@@ -76,4 +102,9 @@
         <xacro:material_yaskawa_blue/>
       </visual>
+      <inertial>
+        <origin xyz="0 0 0" rpy="0 0 0"/>
+        <mass value="0.1"/>
+        <inertia ixx="0.03" ixy="0.03" ixz="0.03" iyy="0.0" iyz="0.0" izz="0.0"/>
+      </inertial>
       <collision>
         <geometry>
@@ -89,4 +120,9 @@
         <xacro:material_yaskawa_blue/>
       </visual>
+      <inertial>
+        <origin xyz="0 0 0" rpy="0 0 0"/>
+        <mass value="0.1"/>
+        <inertia ixx="0.03" ixy="0.03" ixz="0.03" iyy="0.0" iyz="0.0" izz="0.0"/>
+      </inertial>
       <collision>
         <geometry>
@@ -98,4 +134,9 @@
     <!-- end of link list -->
     <!-- joint list -->
+    <joint name="world_fixed" type="fixed">
+      <parent link="world"/>
+      <child link="${prefix}base_link"/>
+      <origin xyz="0 0 0" rpy="0 0 0"/>
+    </joint>
     <joint name="${prefix}joint_1_s" type="revolute">
       <parent link="${prefix}base_link"/>
@@ -104,4 +145,5 @@
       <axis xyz="0 0 1" />
       <limit lower="${radians(-180)}" upper="${radians(180)}" effort="368.48" velocity="${radians(130)}"/>
+      <dynamics damping="1"/>
     </joint>
     <joint name="${prefix}joint_2_l" type="revolute">
@@ -111,4 +153,5 @@
       <axis xyz="0 1 0" />
       <limit lower="${radians(-180)}" upper="${radians(180)}" effort="368.48" velocity="${radians(130)}"/>
+      <dynamics damping="1"/>
     </joint>
     <joint name="${prefix}joint_3_u" type="revolute">
@@ -118,4 +161,5 @@
       <axis xyz="0 -1 0" />
       <limit lower="${radians(-5)}" upper="${radians(355)}" effort="141.12" velocity="${radians(180)}"/>
+      <dynamics damping="1"/>
     </joint>
     <joint name="${prefix}joint_4_r" type="revolute">
@@ -125,4 +169,5 @@
       <axis xyz="0 0 1" />
       <limit lower="${radians(-180)}" upper="${radians(180)}" effort="39.20" velocity="${radians(180)}"/>
+      <dynamics damping="1"/>
     </joint>
     <joint name="${prefix}joint_5_b" type="revolute">
@@ -132,4 +177,5 @@
       <axis xyz="0 -1 0" />
       <limit lower="${radians(-180)}" upper="${radians(180)}" effort="31.36" velocity="${radians(250)}"/>
+      <dynamics damping="1"/>
     </joint>
     <joint name="${prefix}joint_6_t" type="revolute">
@@ -139,4 +185,5 @@
       <axis xyz="0 0 1" />
       <limit lower="${radians(-180)}" upper="${radians(180)}" effort="31.36" velocity="${radians(250)}"/>
+      <dynamics damping="1"/>
     </joint>
     <joint name="${prefix}joint_6_t-tool0" type="fixed">
@@ -154,3 +201,39 @@
     </joint>
   </xacro:macro>
+  <gazebo reference="camera_depth_frame">
+    <sensor name="kinect_camera" type="depth">
+      <update_rate>20</update_rate>
+      <camera>
+        <horizontal_fov>1.047198</horizontal_fov>
+        <image>
+          <width>640</width>
+          <height>480</height>
+          <format>B8G8R8</format>
+        </image>
+        <clip>
+          <near>0.05</near>
+          <far>3</far>
+        </clip>
+      </camera>
+      <plugin name="kinect_controller" filename="libgazebo_ros_openni_kinect.so">
+        <baseline>0.1</baseline>
+        <alwaysOn>true</alwaysOn>
+        <updateRate>10</updateRate>
+        <cameraName>camera_ir</cameraName>
+        <imageTopicName>/camera/color/image_raw</imageTopicName>
+        <cameraInfoTopicName>/camera/color/camera_info</cameraInfoTopicName>
+        <depthImageTopicName>/camera/depth/image_raw</depthImageTopicName>
+        <depthImageCameraInfoTopicName>/camera/depth/camera_info</depthImageCameraInfoTopicName>
+        <pointCloudTopicName>/camera/depth/points</pointCloudTopicName>
+        <frameName>camera_depth_optical_frame</frameName>
+        <distortion_k1>0.0</distortion_k1>
+        <distortion_k2>0.0</distortion_k2>
+        <distortion_k3>0.0</distortion_k3>
+        <distortion_t1>0.0</distortion_t1>
+        <distortion_t2>0.0</distortion_t2>
+        <pointCloudCutoff>0.16</pointCloudCutoff>
+        <pointCloudCutoffMax>10.0</pointCloudCutoffMax>
+      </plugin>
+    </sensor>
+  </gazebo>
 </robot>

Commit message: add hc10 moveif config add edit xacro

File: catkin_ws/src/motoman/motoman_hc10_support/urdf/hc10_macro.xacro (robot description, xacro)
@@ -6,4 +6,9 @@
     <link name="world"/>
     <link name="${prefix}base_link">
+    	<inertial>
+	   	<origin xyz="0 0 0" rpy="0 0 0"/>
+	   	<mass value="0.1"/>
+	   	<inertia ixx="0.03" ixy="0.03" ixz="0.03" iyy="0.0" iyz="0.0" izz="0.0"/>
+	</inertial>
       <visual>
         <geometry>
@@ -12,9 +17,4 @@
         <xacro:material_yaskawa_blue/>
       </visual>
-      <inertial>
-        <origin xyz="0 0 0" rpy="0 0 0"/>
-        <mass value="0.1"/>
-        <inertia ixx="0.03" ixy="0.03" ixz="0.03" iyy="0.0" iyz="0.0" izz="0.0"/>
-      </inertial>
       <collision>
         <geometry>
@@ -24,4 +24,9 @@
     </link>
     <link name="${prefix}link_1_s">
+    	<inertial>
+	   	<origin xyz="0 0 0" rpy="0 0 0"/>
+	   	<mass value="0.1"/>
+	   	<inertia ixx="0.03" ixy="0.03" ixz="0.03" iyy="0.0" iyz="0.0" izz="0.0"/>
+	</inertial>
       <visual>
         <geometry>
@@ -30,9 +35,4 @@
         <xacro:material_yaskawa_blue/>
       </visual>
-      <inertial>
-        <origin xyz="0 0 0" rpy="0 0 0"/>
-        <mass value="0.1"/>
-        <inertia ixx="0.03" ixy="0.03" ixz="0.03" iyy="0.0" iyz="0.0" izz="0.0"/>
-      </inertial>
       <collision>
         <geometry>
@@ -42,4 +42,9 @@
     </link>
     <link name="${prefix}link_2_l">
+    	<inertial>
+	   	<origin xyz="0 0 0" rpy="0 0 0"/>
+	   	<mass value="0.1"/>
+	   	<inertia ixx="0.03" ixy="0.03" ixz="0.03" iyy="0.0" iyz="0.0" izz="0.0"/>
+	</inertial>
       <visual>
         <geometry>
@@ -48,9 +53,4 @@
         <xacro:material_yaskawa_blue/>
       </visual>
-      <inertial>
-        <origin xyz="0 0 0" rpy="0 0 0"/>
-        <mass value="0.1"/>
-        <inertia ixx="0.03" ixy="0.03" ixz="0.03" iyy="0.0" iyz="0.0" izz="0.0"/>
-      </inertial>
       <collision>
         <geometry>
@@ -60,4 +60,9 @@
     </link>
     <link name="${prefix}link_3_u">
+    	<inertial>
+	   	<origin xyz="0 0 0" rpy="0 0 0"/>
+	   	<mass value="0.1"/>
+	   	<inertia ixx="0.03" ixy="0.03" ixz="0.03" iyy="0.0" iyz="0.0" izz="0.0"/>
+	</inertial>
       <visual>
         <geometry>
@@ -66,9 +71,4 @@
         <xacro:material_yaskawa_blue/>
       </visual>
-      <inertial>
-        <origin xyz="0 0 0" rpy="0 0 0"/>
-        <mass value="0.1"/>
-        <inertia ixx="0.03" ixy="0.03" ixz="0.03" iyy="0.0" iyz="0.0" izz="0.0"/>
-      </inertial>
       <collision>
         <geometry>
@@ -78,4 +78,9 @@
     </link>
     <link name="${prefix}link_4_r">
+    	<inertial>
+	   	<origin xyz="0 0 0" rpy="0 0 0"/>
+	   	<mass value="0.1"/>
+	   	<inertia ixx="0.03" ixy="0.03" ixz="0.03" iyy="0.0" iyz="0.0" izz="0.0"/>
+	</inertial>
       <visual>
         <geometry>
@@ -84,9 +89,4 @@
         <xacro:material_yaskawa_blue/>
       </visual>
-      <inertial>
-        <origin xyz="0 0 0" rpy="0 0 0"/>
-        <mass value="0.1"/>
-        <inertia ixx="0.03" ixy="0.03" ixz="0.03" iyy="0.0" iyz="0.0" izz="0.0"/>
-      </inertial>
       <collision>
         <geometry>
@@ -96,4 +96,9 @@
     </link>
     <link name="${prefix}link_5_b">
+    	<inertial>
+	   	<origin xyz="0 0 0" rpy="0 0 0"/>
+	   	<mass value="0.1"/>
+	   	<inertia ixx="0.03" ixy="0.03" ixz="0.03" iyy="0.0" iyz="0.0" izz="0.0"/>
+	</inertial>
       <visual>
         <geometry>
@@ -102,9 +107,4 @@
         <xacro:material_yaskawa_blue/>
       </visual>
-      <inertial>
-        <origin xyz="0 0 0" rpy="0 0 0"/>
-        <mass value="0.1"/>
-        <inertia ixx="0.03" ixy="0.03" ixz="0.03" iyy="0.0" iyz="0.0" izz="0.0"/>
-      </inertial>
       <collision>
         <geometry>
@@ -114,4 +114,9 @@
     </link>
     <link name="${prefix}link_6_t">
+    	<inertial>
+	   	<origin xyz="0 0 0" rpy="0 0 0"/>
+	   	<mass value="0.1"/>
+	   	<inertia ixx="0.03" ixy="0.03" ixz="0.03" iyy="0.0" iyz="0.0" izz="0.0"/>
+	</inertial>
       <visual>
         <geometry>
@@ -120,9 +125,4 @@
         <xacro:material_yaskawa_blue/>
       </visual>
-      <inertial>
-        <origin xyz="0 0 0" rpy="0 0 0"/>
-        <mass value="0.1"/>
-        <inertia ixx="0.03" ixy="0.03" ixz="0.03" iyy="0.0" iyz="0.0" izz="0.0"/>
-      </inertial>
       <collision>
         <geometry>
@@ -132,12 +132,17 @@
     </link>
     <link name="${prefix}tool0"/>
+    	<inertial>
+	   	<origin xyz="0 0 0" rpy="0 0 0"/>
+	   	<mass value="0.1"/>
+	   	<inertia ixx="0.03" ixy="0.03" ixz="0.03" iyy="0.0" iyz="0.0" izz="0.0"/>
+	</inertial>
     <!-- end of link list -->
     <!-- joint list -->
     <joint name="world_fixed" type="fixed">
-      <parent link="world"/>
-      <child link="${prefix}base_link"/>
-      <origin xyz="0 0 0" rpy="0 0 0"/>
-    </joint>
+	   <parent link="world"/>
+	   <child link="${prefix}base"/>
+	</joint>
     <joint name="${prefix}joint_1_s" type="revolute">
+    	<dynamics damping="1"/>
       <parent link="${prefix}base_link"/>
       <child link="${prefix}link_1_s"/>
@@ -145,7 +150,7 @@
       <axis xyz="0 0 1" />
       <limit lower="${radians(-180)}" upper="${radians(180)}" effort="368.48" velocity="${radians(130)}"/>
-      <dynamics damping="1"/>
     </joint>
     <joint name="${prefix}joint_2_l" type="revolute">
+    	<dynamics damping="1"/>
       <parent link="${prefix}link_1_s"/>
       <child link="${prefix}link_2_l"/>
@@ -153,7 +158,7 @@
       <axis xyz="0 1 0" />
       <limit lower="${radians(-180)}" upper="${radians(180)}" effort="368.48" velocity="${radians(130)}"/>
-      <dynamics damping="1"/>
     </joint>
     <joint name="${prefix}joint_3_u" type="revolute">
+    	<dynamics damping="1"/>
       <parent link="${prefix}link_2_l"/>
       <child link="${prefix}link_3_u"/>
@@ -161,7 +166,7 @@
       <axis xyz="0 -1 0" />
       <limit lower="${radians(-5)}" upper="${radians(355)}" effort="141.12" velocity="${radians(180)}"/>
-      <dynamics damping="1"/>
     </joint>
     <joint name="${prefix}joint_4_r" type="revolute">
+    	<dynamics damping="1"/>
       <parent link="${prefix}link_3_u"/>
       <child link="${prefix}link_4_r"/>
@@ -169,7 +174,7 @@
       <axis xyz="0 0 1" />
       <limit lower="${radians(-180)}" upper="${radians(180)}" effort="39.20" velocity="${radians(180)}"/>
-      <dynamics damping="1"/>
     </joint>
     <joint name="${prefix}joint_5_b" type="revolute">
+    	<dynamics damping="1"/>
       <parent link="${prefix}link_4_r"/>
       <child link="${prefix}link_5_b"/>
@@ -177,7 +182,7 @@
       <axis xyz="0 -1 0" />
       <limit lower="${radians(-180)}" upper="${radians(180)}" effort="31.36" velocity="${radians(250)}"/>
-      <dynamics damping="1"/>
     </joint>
     <joint name="${prefix}joint_6_t" type="revolute">
+    	<dynamics damping="1"/>
       <parent link="${prefix}link_5_b"/>
       <child link="${prefix}link_6_t"/>
@@ -185,5 +190,4 @@
       <axis xyz="0 0 1" />
       <limit lower="${radians(-180)}" upper="${radians(180)}" effort="31.36" velocity="${radians(250)}"/>
-      <dynamics damping="1"/>
     </joint>
     <joint name="${prefix}joint_6_t-tool0" type="fixed">
@@ -197,6 +201,6 @@
     <joint name="${prefix}base_link-base" type="fixed">
       <origin xyz="0 0 0.275" rpy="0 0 0"/>
-      <parent link="${prefix}base_link"/>
-      <child link="${prefix}base"/>
+      <parent link="${prefix}base"/>
+      <child link="${prefix}base_link"/>
     </joint>
   </xacro:macro>

Commit message: Included work environment into gazebo

File: catkin_ws/src/motoman/motoman_hc10_support/urdf/hc10_macro.xacro (robot description, xacro)
@@ -200,5 +200,5 @@
     <link name="${prefix}base" />
     <joint name="${prefix}base_link-base" type="fixed">
-      <origin xyz="0 0 0.275" rpy="0 0 0"/>
+      <origin xyz="0 0 0" rpy="0 0 0"/> <!-- Z was 0.275, changed to 0 -->
       <parent link="${prefix}base"/>
       <child link="${prefix}base_link"/>

Commit message: Add cube traj in position

File: catkin_ws/src/motoman/motoman_hc10_support/urdf/hc10_macro.xacro (robot description, xacro)
@@ -200,5 +200,4 @@
     <link name="${prefix}base" />
     <joint name="${prefix}base_link-base" type="fixed">
-      <origin xyz="0 0 0.275" rpy="0 0 0"/>
       <parent link="${prefix}base"/>
       <child link="${prefix}base_link"/>

Commit message: add camera model

File: catkin_ws/src/motoman/motoman_hc10_support/urdf/hc10_macro.xacro (robot description, xacro)
@@ -3,4 +3,10 @@
   <xacro:macro name="motoman_hc10" params="prefix">
     <xacro:include filename="$(find motoman_resources)/urdf/common_materials.xacro"/>
+    <xacro:include filename="$(find motoman_resources)/urdf/kinect_camera.gazebo"/>
+    <gazebo>
+	  <plugin name="gazebo_ros_control" filename="libgazebo_ros_control.so">
+	    <robotNamespace>/MYROBOT</robotNamespace>
+	  </plugin>
+	</gazebo>
     <!-- link list -->
     <link name="world"/>
@@ -137,4 +143,11 @@
 	   	<inertia ixx="0.03" ixy="0.03" ixz="0.03" iyy="0.0" iyz="0.0" izz="0.0"/>
 	</inertial>
+	<link name="${prefix}camera_link">
+		<visual>
+			<geometry>
+				<box size="0.05 0.1 0.04"/>
+			</geometry>
+		</visual>
+	</link>
     <!-- end of link list -->
     <!-- joint list -->
@@ -204,4 +217,10 @@
       <child link="${prefix}base_link"/>
     </joint>
+	<!-- Attach Kinect to the robot end effector -->
+	<joint type="fixed" name="camera_joint">
+		<origin xyz="0.0 0.0 0.02" rpy="0.0 0.0 0.0"/>
+		<child link="camera_link"/>
+		<parent link="${prefix}tool0"/>
+	</joint>
   </xacro:macro>
 </robot>

Commit message: Fixed faulty physics and pose with environment

File: catkin_ws/src/motoman/motoman_hc10_support/urdf/hc10_macro.xacro (robot description, xacro)
@@ -200,5 +200,5 @@
     <link name="${prefix}base" />
     <joint name="${prefix}base_link-base" type="fixed">
-      <origin xyz="0 0 0" rpy="0 0 0"/> <!-- Z was 0.275, changed to 0 -->
+      <origin xyz="0 0 0.02" rpy="0 0 0"/> <!-- Z was 0.275, changed to 0.02 -->
       <parent link="${prefix}base"/>
       <child link="${prefix}base_link"/>

Commit message: wip

File: catkin_ws/src/motoman/motoman_hc10_support/urdf/hc10_macro.xacro (robot description, xacro)
@@ -3,10 +3,11 @@
   <xacro:macro name="motoman_hc10" params="prefix">
     <xacro:include filename="$(find motoman_resources)/urdf/common_materials.xacro"/>
-    <xacro:include filename="$(find motoman_resources)/urdf/kinect_camera.gazebo"/>
+    <xacro:include filename="$(find camera)/urdf/kinect_camera.xacro"/>
+    <xacro:camera_sim />
     <gazebo>
 	  <plugin name="gazebo_ros_control" filename="libgazebo_ros_control.so">
 	    <robotNamespace>/MYROBOT</robotNamespace>
 	  </plugin>
-	</gazebo>
+	  </gazebo>
     <!-- link list -->
     <link name="world"/>
@@ -143,5 +144,5 @@
 	   	<inertia ixx="0.03" ixy="0.03" ixz="0.03" iyy="0.0" iyz="0.0" izz="0.0"/>
 	</inertial>
-	<link name="${prefix}camera_link">
+	<link name="${prefix}camera_depth_frame">
 		<visual>
 			<geometry>
@@ -220,5 +221,5 @@
 	<joint type="fixed" name="camera_joint">
 		<origin xyz="0.0 0.0 0.02" rpy="0.0 0.0 0.0"/>
-		<child link="camera_link"/>
+		<child link="camera_depth_frame"/>
 		<parent link="${prefix}tool0"/>
 	</joint>

Commit message: camera on robot w/ point cloud

File: catkin_ws/src/motoman/motoman_hc10_support/urdf/hc10_macro.xacro (robot description, xacro)
@@ -3,6 +3,6 @@
   <xacro:macro name="motoman_hc10" params="prefix">
     <xacro:include filename="$(find motoman_resources)/urdf/common_materials.xacro"/>
-    <xacro:include filename="$(find camera)/urdf/kinect_camera.xacro"/>
-    <xacro:camera_sim />
+    <xacro:include filename="$(find camera)/urdf/kinect_ros/model_macro.xacro"/>
+  	<xacro:kinect parent_link="${prefix}tool0"/>
     <gazebo>
 	  <plugin name="gazebo_ros_control" filename="libgazebo_ros_control.so">
@@ -144,11 +144,4 @@
 	   	<inertia ixx="0.03" ixy="0.03" ixz="0.03" iyy="0.0" iyz="0.0" izz="0.0"/>
 	</inertial>
-	<link name="${prefix}camera_depth_frame">
-		<visual>
-			<geometry>
-				<box size="0.05 0.1 0.04"/>
-			</geometry>
-		</visual>
-	</link>
     <!-- end of link list -->
     <!-- joint list -->
@@ -218,10 +211,4 @@
       <child link="${prefix}base_link"/>
     </joint>
-	<!-- Attach Kinect to the robot end effector -->
-	<joint type="fixed" name="camera_joint">
-		<origin xyz="0.0 0.0 0.02" rpy="0.0 0.0 0.0"/>
-		<child link="camera_depth_frame"/>
-		<parent link="${prefix}tool0"/>
-	</joint>
   </xacro:macro>
 </robot>

Commit message: Simplify workspace

File: catkin_ws/src/motoman/motoman_hc10_support/urdf/hc10_macro.xacro (robot description, xacro)
@@ -3,6 +3,4 @@
   <xacro:macro name="motoman_hc10" params="prefix">
     <xacro:include filename="$(find motoman_resources)/urdf/common_materials.xacro"/>
-    <xacro:include filename="$(find camera)/urdf/kinect_ros/model_macro.xacro"/>
-  	<xacro:kinect parent_link="${prefix}tool0"/>
     <gazebo>
 	  <plugin name="gazebo_ros_control" filename="libgazebo_ros_control.so">
@@ -11,4 +9,6 @@
 	  </gazebo>
     <!-- link list -->
+    <xacro:include filename="$(find motoman_hc10_support)/urdf/kinect_sensor.xacro"/>
+    <xacro:kinect parent_link="${prefix}tool0"/>
     <link name="world"/>
     <link name="${prefix}base_link">

File: catkin_ws/src/motoman/motoman_hc10_support/urdf/kinect_sensor.xacro (robot description, xacro)
@@ -15,5 +15,5 @@
       <visual name="visual">
         <geometry>
-          <mesh filename="package://camera/urdf/kinect_ros/meshes/kinect.dae" scale="1 1 1"/>
+          <mesh filename="package://motoman_hc10_support/meshes/kinect/kinect.dae" scale="1 1 1"/>
         </geometry>
       </visual>
