Commit message: camera on robot

File: catkin_ws/src/camera/urdf/kinect_ros/model_macro.xacro (robot description, xacro)
@@ -2,62 +2,60 @@
 <robot xmlns:xacro="http://ros.org/wiki/xacro">
 	<xacro:macro name="kinect" params="parent_link">
-		  <link name="link_kinect">
-		    <inertial>
-		      <mass>0.1</mass>
-		    </inertial>
-		    <collision name="collision">
-		      <geometry>
-		        <box>
-		          <size>0.073000 0.276000 0.072000</size>
-		        </box>
-		      </geometry>
-		    </collision>
-		    <visual name="visual">
-		      <geometry>
-		        <mesh>
-		          <uri>model://kinect/meshes/kinect.dae</uri>
-		        </mesh>
-		      </geometry>
-		    </visual>
-		  </link>
-	<gazebo reference="link_kinect">
-    <sensor name="kinect_camera" type="depth">
-        <update_rate>20</update_rate>
-        <camera>
-            <horizontal_fov>1.047198</horizontal_fov>
-            <image>
-                <width>640</width>
-                <height>480</height>
-                <format>B8G8R8</format>
-            </image>
-            <clip>
-                <near>0.05</near>
-                <far>3</far>
-            </clip>
-        </camera>
-        <plugin name="kinect_controller" filename="libgazebo_ros_openni_kinect.so">
-        <baseline>0.1</baseline>
-        <alwaysOn>true</alwaysOn>
-        <updateRate>10</updateRate>
-        <cameraName>camera_ir</cameraName>
-        <imageTopicName>/camera/color/image_raw</imageTopicName>
-        <cameraInfoTopicName>/camera/color/camera_info</cameraInfoTopicName>
-        <depthImageTopicName>/camera/depth/image_raw</depthImageTopicName>
-        <depthImageCameraInfoTopicName>/camera/depth/camera_info</depthImageCameraInfoTopicName>
-        <pointCloudTopicName>/camera/depth/points</pointCloudTopicName>
-        <frameName>camera_depth_optical_frame</frameName>
-        <distortion_k1>0.0</distortion_k1>
-        <distortion_k2>0.0</distortion_k2>
-        <distortion_k3>0.0</distortion_k3>
-        <distortion_t1>0.0</distortion_t1>
-        <distortion_t2>0.0</distortion_t2>
-        <pointCloudCutoff>0.16</pointCloudCutoff>
-        <pointCloudCutoffMax>10.0</pointCloudCutoffMax>
-        </plugin>
-    </sensor>
-	</gazebo>
+    <link name="link_kinect">
+      <inertial>
+        <origin xyz="0 0 0" rpy="0 0 0"/>
+        <mass value="0.1"/>
+        <inertia ixx="0" ixy="0" ixz="0" iyy="0" iyz="0" izz="0"/>
+      </inertial>
+      <collision name="collision">
+        <geometry>
+          <box size="0.073000 0.276000 0.072000"/>
+        </geometry>
+      </collision>
+      <visual name="visual">
+        <geometry>
+          <mesh filename="package://camera/urdf/kinect_ros/meshes/kinect.dae" scale="1 1 1"/>
+        </geometry>
+      </visual>
+    </link>
+    <gazebo reference="link_kinect">
+      <sensor name="kinect_camera" type="depth">
+          <update_rate>20</update_rate>
+          <camera>
+              <horizontal_fov>1.047198</horizontal_fov>
+              <image>
+                  <width>640</width>
+                  <height>480</height>
+                  <format>B8G8R8</format>
+              </image>
+              <clip>
+                  <near>0.05</near>
+                  <far>3</far>
+              </clip>
+          </camera>
+          <plugin name="kinect_controller" filename="libgazebo_ros_openni_kinect.so">
+          <baseline>0.1</baseline>
+          <alwaysOn>true</alwaysOn>
+          <updateRate>10</updateRate>
+          <cameraName>camera_ir</cameraName>
+          <imageTopicName>/camera/color/image_raw</imageTopicName>
+          <cameraInfoTopicName>/camera/color/camera_info</cameraInfoTopicName>
+          <depthImageTopicName>/camera/depth/image_raw</depthImageTopicName>
+          <depthImageCameraInfoTopicName>/camera/depth/camera_info</depthImageCameraInfoTopicName>
+          <pointCloudTopicName>/camera/depth/points</pointCloudTopicName>
+          <frameName>camera_depth_optical_frame</frameName>
+          <distortion_k1>0.0</distortion_k1>
+          <distortion_k2>0.0</distortion_k2>
+          <distortion_k3>0.0</distortion_k3>
+          <distortion_t1>0.0</distortion_t1>
+          <distortion_t2>0.0</distortion_t2>
+          <pointCloudCutoff>0.16</pointCloudCutoff>
+          <pointCloudCutoffMax>10.0</pointCloudCutoffMax>
+          </plugin>
+      </sensor>
+    </gazebo>
 		  <!-- Attach Kinect to the robot end effector -->
 		<joint type="fixed" name="camera_joint">
-			<origin xyz="0.0 0.0 0.02" rpy="0.0 0.0 0.0"/>
+			<origin xyz="0.0 0.0 0.07" rpy="0.0 -1.57 3.14"/>
 			<child link="link_kinect"/>
 			<parent link="${parent_link}"/>

Commit message: point cloud

File: catkin_ws/src/camera/urdf/kinect_ros/model_macro.xacro (robot description, xacro)
@@ -21,5 +21,5 @@
     <gazebo reference="link_kinect">
       <sensor name="kinect_camera" type="depth">
-          <update_rate>20</update_rate>
+          <update_rate>1000</update_rate>
           <camera>
               <horizontal_fov>1.047198</horizontal_fov>
@@ -57,5 +57,5 @@
 		  <!-- Attach Kinect to the robot end effector -->
 		<joint type="fixed" name="camera_joint">
-			<origin xyz="0.0 0.0 0.07" rpy="0.0 -1.57 3.14"/>
+			<origin xyz="0.0 0.0 0.07" rpy="0.0 -1.57 1.57"/>
 			<child link="link_kinect"/>
 			<parent link="${parent_link}"/>
